File: boards/Arcade Controller/arcade_controller.brd (EAGLE design)
At the start: 56 x 50 mm, 38 parts, among them IC1 LM3S5749, J1 DEBUG, J2 1751248, J3 MINI-USB-UX60-MB-5S8, J4 PTSM_1771088, J5 PTSM_1702474, J6 PTSM_1771088, J7 PTSM_1702474, J8 Ser I/O, SW1 Reset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

Commit message: Battery Charger test board
Parts:
- moved LED1 11.5 mm to (40.0, 9.37), turned to 270 degrees
- moved R3 11.5 mm to (40.0, 9.37), turned to 0 degrees
- moved SW1 8.25 mm to (52.5, 11.4), turned to 90 degrees
- moved C8 8.21 mm to (52.9, 10.2), turned to 270 degrees
- moved R7 5.39 mm to (43.8, 10.2), turned to 270 degrees
- moved R2 5.15 mm to (50.6, 10.2), turned to 270 degrees
- moved SW2 4.53 mm to (45.7, 11.4), turned to 90 degrees
- moved J4 0.62 mm to (27.0, 46.6)
- moved J5 0.62 mm to (48.0, 46.6)
- moved J6 0.62 mm to (3.38, 13.0)
- moved J7 0.62 mm to (3.38, 34.0)
- moved J1 0.38 mm to (49.9, 30.7)
- moved J2 0.25 mm to (10.2, 46.1)
Routing:
- net /RESET: track 61.8 -> 41.7 mm
- net /PROG: track 17.1 -> 12.9 mm
- net N$8: track 65.2 -> 69.1 mm
- net VDD: track 124.9 -> 121.2 mm
- net PG0: track 19.7 -> 22.3 mm, vias 0 -> 2
- net PG1: track 18.3 -> 16.7 mm
- net PE7: track 23.7 -> 22.2 mm
- net PE4: track 19.0 -> 20.2 mm
- net N$12: track 25.4 -> 26.5 mm
- net N$11: track 27.0 -> 27.9 mm
- net PG2: track 16.7 -> 15.9 mm
- net N$10: track 28.6 -> 29.3 mm
- net N$9: track 30.1 -> 30.7 mm
- net PG7: track 32.3 -> 32.9 mm
- net PG6: track 32.0 -> 32.6 mm
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