File: boards/LPC1788 Board/lpc1788_board.brd (EAGLE design)
At the start: 85 x 70 mm, 108 parts, among them J1 5VDC, J10 MOLEX_527930570_5PIN_FFC_CONN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, J11 20PIN_10X2_.100IN, J2 SAMTEC_MUSB, J3 JST_2MM_SMT, J4 Console, J5 SMA-J-P-X-ST-EM1, J6 JTAG, J8 NHD-4.3-480272EF, J9 DF12B-50DX_25X2_0.5MM, Q1 MMBT2907, SW1 Reset, SW2 OS102011MA1QS1, U1 LTC3127EMSEPBF, U2 MAX1551EZK+T, U3 LT3497EDDBTRMPBF, U4 AS4C8M16S-128MBIT_SDRAM, U5 S25FL064P, U6 AR1021-RESISTIVE_TOUCH_CONTRO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, U7 LPC177X_8X-208, U8 NUP2202, Y1 12MHz

Commit message: LPC1788 Board Rev 1
Parts:
- moved J6 1.37 mm to (-32.8, 50.7)
- moved R23 1.37 mm to (-31.1, 53.3)
- moved R24 1.37 mm to (-31.1, 52.0)
- moved R25 1.37 mm to (-31.1, 50.7)
- moved R26 1.37 mm to (-31.1, 49.5)
- moved C6 0.46 mm to (13.4, 62.2)
- moved C4 0.30 mm to (10.9, 60.8)
- moved R10 0.30 mm to (32.9, 91.0)
Connections:
- removed net N$30: J11.13, U7.206
- new net GPIO1: J11.15, U7.25
- new net GPIO2: J11.13, U7.18
Routing:
- net N$30: track 33.6 -> 0.00 mm, vias 4 -> 0
- net GPIO1: track 0.00 -> 19.1 mm, vias 0 -> 2
- net GPIO2: track 0.00 -> 18.7 mm, vias 0 -> 2
- net N$34: track 25.0 -> 22.6 mm
- net SPI_SCK: track 59.4 -> 57.0 mm
- net SPI_MOSI: track 58.6 -> 56.4 mm
- net /RESET: track 55.5 -> 56.8 mm
- net SPI_MISO: track 57.4 -> 56.1 mm
- net TCK/SWDCLK: track 18.1 -> 17.4 mm
- net +3V3: track 504.7 -> 504.2 mm, vias 36 -> 37
- net TDO/SWO: track 15.4 -> 14.9 mm
- net TMS/SWDIO: track 17.3 -> 17.8 mm
- net TDI: track 16.8 -> 16.2 mm
- net N$35: track 24.5 -> 23.9 mm
- net SPI_CS: track 56.3 -> 55.8 mm
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Other:
- board text added: "LPC1788 Board Rev 1"
- board text removed: "ADD GND PLANE VIAS"

Commit message: Storing local changes before upgrading to eagle 6.6.0
Parts:
- removed C32: 10uF, rcl:C0402
- removed C37: 330uF, rcl:C1206
- removed J1: 5VDC, Custom:PJ-045
- removed J8: NHD-4.3-480272EF, Custom:FCI_62684-402100ALF
- removed L3: 15uH, rcl:L3225M
- removed LED1: CHG, led:CHIPLED_0603
- removed SW2: OS102011MA1QS1, Custom:OS102011MA1QS1
- removed U5: S25FL064P, Custom:SO3_016
- added CHG, PGOOD: USB, led:CHIPLED_0603
- added D1: (no value), Custom:SOD-323
- added PWR: OS102011MA1QS1, Custom:OS102011MA1QS1
- added Q3: FDN335N, Custom:SUPER-SOT3
- added R34, R36: 10K, rcl:R0402
- added R35: 2.5, rcl:R0402
- added SW3: ISP, Custom:SMT_PUSHBUTTON
- added TH1: (no value), rcl:0204V
- C1: value 10uF -> 18pF
- C10, C3: value 1uF -> 10uF; device rcl:C0402 -> rcl:C0805K
- C11, C9: value 1uF -> 10uF; device rcl:C0805 -> rcl:C0805K
- C12: value 18pF -> 10uF; device rcl:C0603 -> rcl:C0805K
- C13: value 18pF -> 1uF; device rcl:C0603 -> rcl:C0402
- C16: value 0.1uF -> 1uF; device rcl:C0603 -> rcl:C0402
- C2: value 100pF -> 18pF
- C4: value 22uF -> 0.1uF; device rcl:C0805 -> rcl:C0402
- C6: value 100uF -> 0.1uF; device rcl:C1206 -> rcl:C0402
- C7: value 1uF -> 0.1uF
- C8: value 330uF -> 10uF; device rcl:C1206 -> rcl:C0805K
- L1: value 4.7uH -> 3.3uH; device Custom:NR6028 -> Custom:3015
- L2: value 15uH -> 22uH; device rcl:L3225M -> Custom:4012
- R1: value 320k -> 100K
- R11: value 100K -> 4.7K; device rcl:R0603 -> rcl:R0402
- R12, R26, R27: device rcl:R0603 -> rcl:R0402
- R13: value 4.7K -> 1.5K; device rcl:R0603 -> rcl:R0402
- R14, R28: value 10k -> 10K
- R15: value 1.5K -> 39K; device rcl:R0603 -> rcl:R0402
- R2: value 182k -> 10K
- R22: value 10k -> 24K
- R23: value 10K -> 0; device rcl:R0603 -> rcl:R0402
- R24, R25: value 10K -> 1.5K; device rcl:R0603 -> rcl:R0402
- R29: value 4.7K -> 3.57K; device rcl:R0603 -> rcl:R0402
- R3: value 32.4k -> 10K
- R30: value 4.7K -> 2.94K; device rcl:R0603 -> rcl:R0402
- R32: value 24K -> 4.32K; device rcl:R0603 -> rcl:R0402
- R33: value 39K -> 56.2K; device rcl:R0603 -> rcl:R0402
- R4: value 50 -> 10K
- R5: value 499k -> 10K
- R6: value 10 -> 100K
- R7: value 10 -> 10K
- R8, R9: value 10K -> 4.7K
- U1: value LTC3127EMSEPBF -> BQ24232H-BATTERY_CHARGER; device LTC:SOP65P490X110-13N -> Custom:QFN-16
- U2: value MAX1551EZK+T -> TPS63001-BUCK-BOOST_CONVERTER; device Maxim:SOT95P275X110-5N -> Custom:QFN-10
- U3: value LT3497EDDBTRMPBF -> AP5724; device LTC:DFN300X200X80-11N -> Custom:SOT-26
- moved R22 175.4 mm to (-77.6, -84.1), flipped to the top, turned to 0 degrees
- moved R9 170.9 mm to (-77.6, -59.7)
- moved R8 168.4 mm to (-77.6, -54.9)
- moved R7 160.0 mm to (-77.6, -50.0), turned to 0 degrees
- moved R13 155.6 mm to (-77.6, -74.4), flipped to the top, turned to 0 degrees
- moved R6 155.5 mm to (-77.6, -40.2), turned to 0 degrees
- moved R15 153.0 mm to (-77.6, -79.2), flipped to the top, turned to 0 degrees
- moved R12 150.6 mm to (-77.6, -69.5), flipped to the top, turned to 0 degrees
- moved R4 148.4 mm to (-77.6, -30.5), flipped to the top
- moved R1 139.7 mm to (-77.6, -45.1)
- moved R5 133.6 mm to (-77.6, -35.4), turned to 0 degrees
- moved R3 132.0 mm to (-77.6, -25.6), flipped to the top, turned to 0 degrees
- moved R11 129.4 mm to (-77.6, -64.6), flipped to the top, turned to 0 degrees
- moved R2 123.8 mm to (-77.6, -20.7), flipped to the top, turned to 0 degrees
- moved C2 117.2 mm to (-77.6, -11.0), turned to 0 degrees
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Connections:
- removed net +VBAT: C1.1, C10.1, C37.1, C7.1, L2.1, L3.1, R4.2, R8.2, SW2.P$3, U1.3, U1.4, U2.5, U3.8
- removed net LED1_PWR: J8.P$2, J9.P$30, J9.P$32, R6.1, U3.1
- removed net LED2_PWR: J9.P$36, J9.P$38, R7.1, U3.5
- removed net N$20: J3.2, SW2.P$2
- removed net SPI_FLASH_CS: U5.P$7, U7.130
- removed net SPI_FLASH_MISO: U5.P$8, U7.126
- removed net SPI_FLASH_MOSI: U5.P$15, U7.124
- removed net SPI_FLASH_SCK: U5.P$16, U7.128
- removed net V+: C3.1, J1.1, U2.4
- new net /RESET1: C6.1, R1.1, SW3.P$1, SW3.P$2, U7.110
- new net LED_A: C16.1, D1.C, J9.P$30, J9.P$32, U3.5
- new net LED_K: J9.P$36, J9.P$38, R35.2, U3.3
- new net N$10: R34.1, TH1.2, U1.1
- new net N$14: C10.1, PWR.P$3, U2.5, U2.6, U2.7, U2.8
- new net N$19: R33.2, U1.14
- new net N$30: L1.1, U2.4
- new net N$9: C3.1, J3.2, U1.2, U1.3
- new net SD_PWR: Q3.1, U7.118
- net +3V3: now also C11.1, C12.1, C13.1, L2.1, Q3.3, R12.2, R2.2, R3.2, R4.2, R6.2, R7.2, R8.2, R9.2, U2.1, U2.10, U3.6; no longer C4.1, C6.1, C8.1, J8.P$4, R12.1, R13.1, R22.1, R25.1, R26.1, R27.1, R28.1, R29.1, R30.1, U$3.VDD, U1.10, U5.P$2
- net +VUSB: now also R15.2, R22.2, U1.13; no longer C32.1, R32.1, R33.1, U2.1
- net /RESET: now also C4.1, R6.1; no longer C16.1, R11.1
- net B0: no longer J8.P$21
- net B1: no longer J8.P$22
- net B2: no longer J8.P$23
- net B3: no longer J8.P$24
- net B4: no longer J8.P$25
- net B5: no longer J8.P$26
- net B6: no longer J8.P$27
- net B7: no longer J8.P$28
- net G0: no longer J8.P$13
- net G1: no longer J8.P$14
- net G2: no longer J8.P$15
- net G3: no longer J8.P$16
- net G4: no longer J8.P$17
- net G5: no longer J8.P$18
- net G6: no longer J8.P$19
- net G7: no longer J8.P$20
- net GND: now also R15.1, R27.1, R28.2, R29.1, R30.1, R32.1, R33.1, R34.2, R35.1, R36.1, SW3.P$3, SW3.P$4, TH1.1, U1.4, U1.8, U2.3, U2.9, U3.2; no longer C32.2, C37.2, J1.2, J1.3, J8.P$1, J8.P$29, J8.P$3, J8.P$36, R2.1, R24.2, R3.1, R33.2, R9.1, U1.1, U1.12, U1.13, U1.5, U1.7, U2.2, U3.11, U3.3, U5.P$10
- net KEY_I2C_SCL: now also R11.1; no longer R30.2
- net KEY_I2C_SDA: now also R12.1; no longer R29.2
- net LCD_DCLK: no longer J8.P$30
- net LCD_ENAB_M: no longer J8.P$34
- net LCD_FP: no longer J8.P$33
- net LCD_LP: no longer J8.P$32
- net LCD_PWR: no longer J8.P$31
- net LED_CTRL: now also R36.2; no longer R8.1, R9.2, U3.2
- net N$1: now also C7.1, C8.1, Q3.2, R23.2, R28.1, U$3.VDD; no longer R3.2, U1.6
- net N$11: now also R29.2, U1.15; no longer C11.1, R7.2, U3.6
- net N$12: now also R30.2, U1.12; no longer L2.2, U3.9
- net N$13: now also R32.2, U1.16; no longer L3.2, U3.7
- net N$15: now also C1.1; no longer C12.1
- net N$16: now also C2.1; no longer C13.1
- net N$2: now also C9.1, PWR.P$2, R24.2, R25.2, R26.1, U1.10, U1.11; no longer R1.1, R2.2, U1.8
- net N$21: now also R13.2; no longer R15.2
- net N$25: now also U7.202; no longer U7.94
- net N$26: now also U7.204; no longer U7.96
- net N$3: now also R26.2, U1.5; no longer L1.2, U1.2
- net N$31: now also L1.2, U2.2; no longer R22.2, U5.P$9
- net N$33: now also D1.A, L2.2, U3.1; no longer R28.2, U5.P$1
- net N$35: no longer J8.P$39
- net N$36: no longer J8.P$37
- net N$37: no longer J8.P$38
- net N$38: no longer J8.P$40
- net N$4: now also R27.2, U1.6; no longer L1.1, U1.11
- net N$42: now also R22.1; no longer R32.2
- net N$5: now also PGOOD.A, R24.1; no longer LED1.C, U2.3
- net N$6: now also CHG.A, R25.1; no longer C9.1, R6.2, U3.10
- net N$7: now also PGOOD.C, U1.7; no longer C2.1, R5.2, U1.9
- net N$8: now also CHG.C, U1.9; no longer LED1.A, R4.1
- net R0: no longer J8.P$5
- net R1: no longer J8.P$6
- net R2: no longer J8.P$7
- net R3: no longer J8.P$8
- net R4: no longer J8.P$9
- net R5: no longer J8.P$10
- net R6: no longer J8.P$11
- net R7: no longer J8.P$12
- net SCL: now also R8.1; no longer R12.2
- net SDA: now also R9.1; no longer R13.2
- net TCK/SWDCLK: now also R5.2; no longer R24.1
- net TDI: now also R4.1; no longer R26.2
- net TDO/SWO: now also R3.1; no longer R25.2
- net TMS/SWDIO: now also R2.1; no longer R23.2
- net TRST: now also R7.1; no longer R27.2
- net USB_D_P: now also R13.1; no longer R15.1
Routing:
- net +3V3: track 504.2 -> 397.8 mm, vias 37 -> 31
- net G3: track 85.9 -> 0.00 mm, vias 4 -> 0
- net G2: track 83.9 -> 0.00 mm, vias 4 -> 0
- net B4: track 77.1 -> 0.00 mm, vias 3 -> 0
- net LED1_PWR: track 76.5 -> 0.00 mm, vias 5 -> 0
- net LED2_PWR: track 73.9 -> 0.00 mm, vias 4 -> 0
- net B5: track 73.6 -> 0.00 mm, vias 3 -> 0
- net B6: track 72.9 -> 0.00 mm, vias 3 -> 0
- net B7: track 71.4 -> 0.00 mm, vias 3 -> 0
- net G7: track 71.0 -> 0.00 mm, vias 2 -> 0
- net G6: track 69.8 -> 0.00 mm, vias 2 -> 0
- net G5: track 69.6 -> 0.00 mm, vias 4 -> 0
- net R7: track 68.1 -> 0.00 mm, vias 4 -> 0
- net R6: track 68.1 -> 0.00 mm, vias 4 -> 0
- net G4: track 67.9 -> 0.00 mm, vias 4 -> 0
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- removed copper zone on layer 1, net N$59
Other:
- board text added: "LPC1788 Board Rev 2"
- board text removed: "LPC1788 Board Rev 1"

Commit message: updates
Parts:
- removed J11: 20PIN_10X2_.100IN, Custom:20-PIN_10X2_.100IN
- removed J5: SMA-J-P-X-ST-EM1, Custom:SMA-J-P-X-ST-EM1
- added 3V3, LED_CTRL, TP1, TP10, TP2, TP3, TP4, TP5, TP6, TP7, TP8, TP9, VSYS, VUSB: TPTP10R, testpad:TP10R
- moved R13 161.0 mm to (56.4, 15.0), turned to 90 degrees
- moved R22 151.6 mm to (43.2, 7.47), flipped to the bottom, turned to 180 degrees
- moved R9 148.3 mm to (52.7, 11.1), flipped to the bottom, turned to 90 degrees
- moved R15 147.9 mm to (43.2, 6.10), flipped to the bottom, turned to 180 degrees
- moved R8 144.7 mm to (51.2, 11.1), flipped to the bottom, turned to 90 degrees
- moved R12 132.2 mm to (-9.45, 43.8), turned to 180 degrees
- moved C1 127.0 mm to (49.4, 2.90), turned to 180 degrees
- moved R11 126.9 mm to (-9.45, 42.5), turned to 180 degrees
- moved R7 123.8 mm to (27.4, 15.7), flipped to the bottom, turned to 90 degrees
- moved C2 122.1 mm to (43.7, 2.90)
- moved R6 120.3 mm to (34.7, 2.76), flipped to the bottom, turned to 90 degrees
- moved C4 116.0 mm to (36.9, 2.76), flipped to the bottom, turned to 90 degrees
- moved R1 115.3 mm to (27.3, 2.76), flipped to the bottom, turned to 270 degrees
- moved C6 103.4 mm to (25.5, 2.76), flipped to the bottom, turned to 270 degrees
- moved SW3 103.0 mm to (26.4, 3.96)
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Connections:
- removed net N$27: J5.1, U7.12
- removed net N$32: J11.7, U7.30
- removed net N$34: J11.5, U7.9
- net +3V3: now also 3V3.TP; no longer J11.1, J11.2, J11.3, J11.4
- net +VUSB: now also VUSB.TP
- net B0: now also J9.P$7; no longer J9.P$11
- net B1: now also J9.P$9; no longer J9.P$13
- net B2: now also J9.P$31; no longer J9.P$8
- net B3: now also J9.P$33; no longer J9.P$6
- net B4: now also J9.P$41; no longer J9.P$37
- net B6: now also J9.P$37; no longer J9.P$41
- net B7: now also J9.P$35; no longer J9.P$43
- net EXT_UART_RX: no longer J11.16
- net EXT_UART_TX: no longer J11.14
- net G0: now also J9.P$18; no longer J9.P$15
- net G2: now also J9.P$24; no longer J9.P$22
- net G3: now also J9.P$26; no longer J9.P$24
- net G4: now also J9.P$40; no longer J9.P$16
- net G5: now also J9.P$42; no longer J9.P$14
- net G6: now also J9.P$44; no longer J9.P$12
- net G7: now also J9.P$46; no longer J9.P$10
- net GND: no longer J11.17, J11.18, J11.19, J11.20, J5.G@1, J5.G@2, J5.G@3, J5.G@4
- net GPIO1: no longer J11.15
- net GPIO2: no longer J11.13
- net KEY_I2C_SCL: no longer U7.141
- net KEY_I2C_SDA: no longer U7.117
- net LCD_DCLK: now also J9.P$15; no longer J9.P$21
- net LCD_ENAB_M: now also J9.P$19; no longer J9.P$25
- net LCD_FP: now also J9.P$17; no longer J9.P$23
- net LCD_LE: now also J9.P$13; no longer J9.P$19
- net LCD_LP: now also J9.P$21; no longer J9.P$27
- net LCD_PWR: now also J9.P$11; no longer J9.P$17
- net LED_A: now also J9.P$6, J9.P$8; no longer J9.P$30, J9.P$32
- net LED_CTRL: now also LED_CTRL.TP, TP4.TP
- net LED_K: now also J9.P$12, J9.P$14; no longer J9.P$36, J9.P$38
- net N$2: now also VSYS.TP
- net N$35: now also J9.P$34
- net N$36: now also J9.P$32
- net N$37: now also J9.P$30
- net N$38: now also J9.P$28
- net R0: now also J9.P$22; no longer J9.P$9
- net R1: now also J9.P$20; no longer J9.P$7
- net R2: now also J9.P$27; no longer J9.P$33
- net R3: now also J9.P$29; no longer J9.P$35
- net R4: now also J9.P$23; no longer J9.P$29
- net R5: now also J9.P$25; no longer J9.P$31
- net R6: now also J9.P$36; no longer J9.P$18
- net R7: now also J9.P$38; no longer J9.P$20
- net SCL: now also R9.1; no longer J11.11, R8.1
- net SDA: now also R8.1; no longer J11.9, R9.1
- net SD_CLK: now also TP1.TP
- net SD_CMD: now also TP2.TP
- net SD_DAT_0: now also TP9.TP
- net SD_DAT_1: now also TP5.TP
- net SD_DAT_2: now also TP7.TP
- net SD_DAT_3: now also TP8.TP
- net SD_PWR: now also TP3.TP
- net SPI_CS: now also TP6.TP; no longer J11.12
- net SPI_MISO: no longer J11.10
- net SPI_MOSI: no longer J11.8
- net SPI_SCK: no longer J11.6
Routing:
- net KEY_INT: track 113.5 -> 8.61 mm, vias 3 -> 2
- net SDA: track 90.1 -> 0.00 mm, vias 3 -> 0
- net SCL: track 86.8 -> 0.00 mm, vias 2 -> 0
- net /RESET1: track 0.00 -> 65.6 mm, vias 0 -> 4
- net EXT_UART_RX: track 57.2 -> 0.00 mm, vias 1 -> 0
- net SPI_SCK: track 57.0 -> 0.00 mm, vias 1 -> 0
- net EXT_UART_TX: track 56.7 -> 0.00 mm, vias 1 -> 0
- net SPI_MOSI: track 56.4 -> 0.00 mm, vias 1 -> 0
- net SPI_MISO: track 56.1 -> 0.00 mm, vias 1 -> 0
- net SPI_CS: track 55.8 -> 0.00 mm, vias 1 -> 0
- net LED_CTRL: track 55.5 -> 2.74 mm, vias 2 -> 1
- net R6: track 0.00 -> 52.3 mm
- net R7: track 0.00 -> 49.3 mm
- net +3V3: track 397.8 -> 348.7 mm, vias 31 -> 41
- net G4: track 0.00 -> 47.1 mm
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- added copper zone on layer 1, net KEEPOUT
- added copper zone on layer 1, net N$14
- added copper zone on layer 1, net N$20
- added copper zone on layer 16, net N$9
- removed copper zone on layer 1, net +VBAT
- removed copper zone on layer 16, net +VBAT
- removed copper zone on layer 16, net N$20
Other:
- board size 85 x 70 mm -> 85 x 57.1 mm
