File: boards/LPC1788 Board/lpc1788_board.sch (EAGLE design)
At the start: 59 parts, among them J1 5VDC, J2 SAMTEC_MUSB, J3 JST_2MM_SMT, J5 SMA-J-P-X-ST-EM1, Q1 MMBT2907, SW1 Reset, U1 LTC3127EMSEPBF, U2 MAX1551EZK+T, U3 LT3497EDDBTRMPBF, U4 CY62167_16MBIT_SRAM, X1 12MHz

Commit message: Continued work on LPC1788 board
Parts:
- removed JP1: RESISTOR_JUMPER_0402, Custom:RESISTOR_JUMPER_0402
- removed R10, R9: 0, rcl:R-US_R0402
- removed U$2: NHD-3.5-320240MF, Custom:NHD-3.5-320240MF
- added C19, C20, C21, C22, C23, C24, C25, C26, C27, C28, C29, C30, C31: 0.1uF, rcl:C-EUC0402
- added C32: 10uF, rcl:C-EUC0402
- added J10: MOLEX_527930570_5PIN_FFC_CONNECTOR, Custom:MOLEX_527930570_5PIN_FFC_CONNECTOR
- added J11: 20PIN_10X2_.100IN, Custom:20PIN_10X2_.100IN
- added J12, J9: DF12B-50DX_25X2_0.5MM, Custom:DF12B-50DX_25X2_0.5MM
- added J6: JTAG, Custom:10PIN_5X2_.050IN
- added J7: JTAG, Custom:8PIN_SIP_.100IN
- added J8: NHD-4.3-480272EF, Custom:NHD-4.3-480272EF
- added R12, R13, R29, R30: 4.7K, rcl:R-US_R0603
- added R21: 0, rcl:R-US_R0603
- added R22, R28: 10k, rcl:R-US_R0402
- added R23, R24, R25, R26, R27: 10K, rcl:R-US_R0603
- added U$4: NUP2202, Custom:NUP2202
- added U5: S25FL064P, Custom:S25FL064P
- C14, C15: value 100nF -> 0.1uF
- C16: value .1uF -> 0.1uF
- J4: value (none) -> Console
- LED2: value CHG -> USB
- R8: value 0 -> 10K
- renumbered X1 to Y1
Connections:
- removed net LED+1: JP1.2, U$2.LED+1
- removed net LED-: U$2.LED-, U$2.LED-1, U$2.VSS, U$2.VSS@1
- removed net N$10: R9.2, U$2.NC
- removed net N$14: R10.2, U$2.NC@1
- removed net N$19: J2.2, R18.1
- removed net N$20: J2.3, R17.1
- removed net N$9: R8.2, U$2.DE
- removed net USB_D+: C17.1, R15.1, R17.2
- removed net USB_D-: C18.1, R18.2
- new net !CS1: U$1PORT4.P4[31]/!EMC_CS1!
- new net D_N: J2.2, R18.1, U$4.P$6
- new net D_P: J2.3, R17.1, U$4.P$1
- new net EXT_UART_RX: J11.S16, U$1PORT0.P0[11]/U2_RXD/I2C2_SCL/T3_MAT1
- new net EXT_UART_TX: J11.S14, U$1PORT0.P0[10]/U2_TXD/I2C2_SDA/T3_MAT0
- new net KEY_I2C_SCL: J10.S3, R30.2, U$1PORT0.P0[28]/I2C0_SCL/USB_SCL1
- new net KEY_I2C_SDA: J10.S2, R29.2, U$1PORT0.P0[27]/I2C0_SDA/USB_SDA1
- new net KEY_INT: J10.S4, U$1PORT0.P0[29]/USB_D+1/EINT_0
- new net N$30: J11.S13, U$1PORT5.P5[4]/U0_OE/T3_MAT3/U4_TXD
- new net N$31: R22.2, U5.W#/ACC/IO2
- new net N$32: J11.S7, U$1PORT5.P5[1]/EMC_A[25]/T2_MAT3
- new net N$33: R28.2, U5.HOLD#/IO3
- new net N$34: J11.S5, U$1PORT5.P5[0]/EMC_A[24]/T2_MAT2
- new net N$36: J7.S1, R21.1
- new net SCL: J11.S11, R13.2, U$1PORT5.P5[3]/U4_RXD/I2C0_SCL
- new net SDA: J11.S9, R12.2, U$1PORT5.P5[2]/T3_MAT2/I2C0_SDA
- new net SPI_CS: J11.S12, U$1PORT1.P1[8]/ENET_CRS/T3_MAT1/SSP2_SSEL
- new net SPI_FLASH_CS: U$1PORT0.P0[16]/U1_RXD/SSP0_SSEL, U5.CS#
- new net SPI_FLASH_MISO: U$1PORT0.P0[17]/U1_CTS/SSP0_MISO, U5.SO/IO1
- new net SPI_FLASH_MOSI: U$1PORT0.P0[18]/U1_DCD/SSP0_MOSI, U5.SI/IO0
- new net SPI_FLASH_SCK: U$1PORT0.P0[15]/U1_TXD/SSP0_SCK, U5.SCK
- new net SPI_MISO: J11.S10, U$1PORT1.P1[4]/ENET_TX_EN/T3_MAT2/SSP2_MISO
- new net SPI_MOSI: J11.S8, U$1PORT1.P1[1]/ENET_TXD1/T3_MAT3/SSP2_MOSI
- new net SPI_SCK: J11.S6, U$1PORT1.P1[0]/ENET_TXD0/T3_CAP1/SSP2_SCK
- new net TCK/SWDCLK: J6.S4, J7.S3, R24.1, U$1MAIN.JTAG_TCK(SWDCLK)
- new net TDI: J6.S8, J7.S5, R26.2, U$1MAIN.JTAG_TDI
- new net TDO/SWO: J6.S6, J7.S4, R25.2, U$1MAIN.JTAG_TDO(SWO)
- new net TMS/SWDIO: J6.S2, J7.S2, R23.2, U$1MAIN.JTAG_TMS(SWDIO)
- new net TRST: R27.2, U$1MAIN.!JTAG_TRST!
- new net USB_D_N: C18.1, R18.2, U$1PORT0.USB_D-2
- new net USB_D_P: C17.1, R15.1, R17.2, U$1PORT0.P0[31]/USB_D+2
- net !BLS0: now also U$1PORT4.P4[26]/!EMC_BLS0!
- net !BLS1: now also U$1PORT4.P4[27]/!EMC_BLS1!
- net !CS0: now also U$1PORT4.P4[30]/!EMC_CS0!
- net !OE: now also U$1PORT4.P4[24]/!EMC_OE!
- net !WE: now also U$1PORT4.P4[25]/!EMC_WE!
- net +3V3: now also C19.1, C20.1, C21.1, C22.1, C23.1, C24.1, C25.1, C26.1, C27.1, C28.1, C29.1, C30.1, C31.1, J10.S1, J11.S1, J11.S2, J11.S3, J11.S4, J12.S1, J12.S2, J6.S1, J8.VDD, J9.S1, J9.S2, R12.1, R13.1, R21.2, R22.1, R23.1, R25.1, R26.1, R27.1, R28.1, R29.1, R30.1, U5.VCC; no longer U$2.VDD, U$2.VDD@1
- net +VUSB: now also C32.1, U$4.P$5
- net /RESET: now also J6.S10, J7.S6, U$1MAIN.!RESET!
- net A0: now also U$1PORT4.P4[0]/EMC_A[0]
- net A1: now also U$1PORT4.P4[1]/EMC_A[1]
- net A10: now also U$1PORT4.P4[10]/EMC_A[10]
- net A11: now also U$1PORT4.P4[11]/EMC_A[11]
- net A12: now also U$1PORT4.P4[12]/EMC_A[12]
- net A13: now also U$1PORT4.P4[13]/EMC_A[13]
- net A14: now also U$1PORT4.P4[14]/EMC_A[14]
- net A15: now also U$1PORT4.P4[15]/EMC_A[15]
- net A16: now also U$1PORT4.P4[16]/EMC_A[16]
- net A17: now also U$1PORT4.P4[17]/EMC_A[17]
- net A18: now also U$1PORT4.P4[18]/EMC_A[18]
- net A19: now also U$1PORT4.P4[19]/EMC_A[19]
- net A2: now also U$1PORT4.P4[2]/EMC_A[2]
- net A3: now also U$1PORT4.P4[3]/EMC_A[3]
- net A4: now also U$1PORT4.P4[4]/EMC_A[4]
- net A5: now also U$1PORT4.P4[5]/EMC_A[5]
- net A6: now also U$1PORT4.P4[6]/EMC_A[6]
- net A7: now also U$1PORT4.P4[7]/EMC_A[7]
- net A8: now also U$1PORT4.P4[8]/EMC_A[8]
- net A9: now also U$1PORT4.P4[9]/EMC_A[9]
- net B0: now also J8.B0; no longer U$2.B0
- net B1: now also J8.B1; no longer U$2.B1
- net B2: now also J8.B2; no longer U$2.B2
- net B3: now also J8.B3; no longer U$2.B3
- net B4: now also J8.B4; no longer U$2.B4
- net B5: now also J8.B5; no longer U$2.B5
- net B6: now also J8.B6; no longer U$2.B6
- net B7: now also J8.B7; no longer U$2.B7
- net D0: now also U$1PORT3.P3[0]/EMC_D[0]
- net D1: now also U$1PORT3.P3[1]/EMC_D[1]
- net D10: now also U$1PORT3.P3[10]/EMC_D[10]
- net D11: now also U$1PORT3.P3[11]/EMC_D[11]
- net D12: now also U$1PORT3.P3[12]/EMC_D[12]
- net D13: now also U$1PORT3.P3[13]/EMC_D[13]
- net D14: now also U$1PORT3.P3[14]/EMC_D[14]
- net D15: now also U$1PORT3.P3[15]/EMC_D[15]
- net D2: now also U$1PORT3.P3[2]/EMC_D[2]
- net D3: now also U$1PORT3.P3[3]/EMC_D[3]
- net D4: now also U$1PORT3.P3[4]/EMC_D[4]
- net D5: now also U$1PORT3.P3[5]/EMC_D[5]
- net D6: now also U$1PORT3.P3[6]/EMC_D[6]
- net D7: now also U$1PORT3.P3[7]/EMC_D[7]
- net D8: now also U$1PORT3.P3[8]/EMC_D[8]
- net D9: now also U$1PORT3.P3[9]/EMC_D[9]
- net G0: now also J8.G0; no longer U$2.G0
- net G1: now also J8.G1; no longer U$2.G1
- net G2: now also J8.G2; no longer U$2.G2
- net G3: now also J8.G3; no longer U$2.G3
- net G4: now also J8.G4; no longer U$2.G4
- net G5: now also J8.G5; no longer U$2.G5
- net G6: now also J8.G6; no longer U$2.G6
- net G7: now also J8.G7; no longer U$2.G7
- net GND: now also C19.2, C20.2, C21.2, C22.2, C23.2, C24.2, C25.2, C26.2, C27.2, C28.2, C29.2, C30.2, C31.2, C32.2, J10.S5, J11.S17, J11.S18, J11.S19, J11.S20, J12.S49, J12.S50, J6.S3, J6.S5, J6.S9, J7.S8, J8.GND, J8.GND@1, J8.GND@2, J8.LED-, J9.S49, J9.S50, R24.2, U$4.P$2, U5.GND
- net LCD_DCLK: now also J8.CLK; no longer U$2.DCLK
- net LCD_ENAB_M: now also J8.DE; no longer R8.1
- net LCD_FP: now also J8.VSYNC; no longer U$2.VSYNC
- net LCD_LE: no longer R9.1
- net LCD_LP: now also J8.HSYNC; no longer U$2.HSYNC
- net LCD_PWR: now also J8.DISP; no longer R10.1
- net LED1_PWR: now also J8.LED+; no longer JP1.1, U$2.LED+
- net LED2_PWR: no longer JP1.3
- net LED_CTRL: now also U$1PORT1.P1[2]/ENET_TXD2/SD_CLK/PWM0_1
- net R0: now also J8.R0; no longer U$2.R0
- net R1: now also J8.R1; no longer U$2.R1
- net R2: now also J8.R2; no longer U$2.R2
- net R3: now also J8.R3; no longer U$2.R3
- net R4: now also J8.R4; no longer U$2.R4
- net R5: now also J8.R5; no longer U$2.R5
- net R6: now also J8.R6; no longer U$2.R6
- net R7: now also J8.R7; no longer U$2.R7
Other:
- note added: "Button Interface"
- note added: "Expansion Interface"
- note added: "JTAG"
- note added: "LPC-LINK"
- note added: "MicroSD Card"
- note added: "Programming and Debug"
- note added: "Reverse add pins to LCD header"
- note added: "Reverse add pins to mem header"
- note added: "SPI Flash"
- note removed: "Add NUP2202 TVS for USB"
- note removed: "Add decoupling caps"
- note removed: "Add header for JTAG"
- note removed: "For NHD-3.5-320240MF No stuff R8-R10 Single supply backlight: Stuff JP1 as 1-2 Dual supply backlight: Stuff JP1 as 2-3"

Commit message: more lpc1788 board changes
Parts:
- added R9: 10K, rcl:R-US_R0402
Connections:
- new net !CAS: J12.S48, U$1PORT2.P2[16]/!EMC_CAS!
- new net !DYCS0: J12.S39, U$1PORT2.P2[20]/!EMC_DYCS0!
- new net !RAS: J12.S49, U$1PORT2.P2[17]/!EMC_RAS!
- new net CKE: J12.S43, U$1PORT2.P2[24]/EMC_CKE0
- new net CLK: J12.S41, U$1PORT2.P2[18]/EMC_CLK[0]
- new net DQM0: J12.S45, U$1PORT2.P2[28]/EMC_DQM0
- new net DQM1: J12.S47, U$1PORT2.P2[29]/EMC_DQM1
- net !BLS0: now also J12.S44
- net !BLS1: now also J12.S46
- net !CS1: now also J12.S42
- net !OE: now also J12.S35
- net !WE: now also J12.S37
- net +3V3: no longer J12.S2
- net +VBAT: now also R8.2
- net A0: now also J12.S2
- net A1: now also J12.S4
- net A10: now also J12.S22
- net A11: now also J12.S24
- net A12: now also J12.S26
- net A13: now also J12.S28
- net A14: now also J12.S30
- net A15: now also J12.S32
- net A16: now also J12.S34
- net A17: now also J12.S36
- net A18: now also J12.S38
- net A19: now also J12.S40
- net A2: now also J12.S6
- net A3: now also J12.S8
- net A4: now also J12.S10
- net A5: now also J12.S12
- net A6: now also J12.S14
- net A7: now also J12.S16
- net A8: now also J12.S18
- net A9: now also J12.S20
- net B0: now also J9.S9
- net B1: now also J9.S11
- net B2: now also J9.S13
- net B3: now also J9.S15
- net B4: now also J9.S17
- net B5: now also J9.S19
- net B6: now also J9.S21
- net B7: now also J9.S23
- net D0: now also J12.S3
- net D1: now also J12.S5
- net D10: now also J12.S23
- net D11: now also J12.S25
- net D12: now also J12.S27
- net D13: now also J12.S29
- net D14: now also J12.S31
- net D15: now also J12.S33
- net D2: now also J12.S7
- net D3: now also J12.S9
- net D4: now also J12.S11
- net D5: now also J12.S13
- net D6: now also J12.S15
- net D7: now also J12.S17
- net D8: now also J12.S19
- net D9: now also J12.S21
- net G0: now also J9.S10
- net G1: now also J9.S12
- net G2: now also J9.S14
- net G3: now also J9.S16
- net G4: now also J9.S18
- net G5: now also J9.S20
- net G6: now also J9.S22
- net G7: now also J9.S24
- net GND: now also R9.1; no longer J12.S49
- net LCD_DCLK: now also J9.S5
- net LCD_ENAB_M: now also J9.S7
- net LCD_FP: now also J9.S8
- net LCD_LE: now also J9.S4
- net LCD_LP: now also J9.S6
- net LCD_PWR: now also J9.S3
- net LED1_PWR: now also J9.S26
- net LED2_PWR: now also J9.S28
- net LED_CTRL: now also R8.1, R9.2
- net R0: now also J9.S25
- net R1: now also J9.S27
- net R2: now also J9.S29
- net R3: now also J9.S31
- net R4: now also J9.S33
- net R5: now also J9.S35
- net R6: now also J9.S37
- net R7: now also J9.S39
Other:
- note added: "Populate either R8 or R9 R8=Normally On R9=Normally Off"
- note removed: "Reverse add pins to LCD header"
- note removed: "Reverse add pins to mem header"
- moved on the sheet: C10, C11, C17, C18, C3, C32, C5, C7, C9, J1, J2, J3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

Commit message: more layout of LPC1788 board
Parts:
- removed J7: JTAG, Custom:8PIN_SIP_.100IN
- removed R21: 0, rcl:R-US_R0603
- added SW2: OS102011MA1QS1, Custom:OS102011MA1QS1
Connections:
- removed net N$36: J7.S1, R21.1
- new net N$20: J3.+, SW2.P
- net +3V3: no longer R21.2
- net +VBAT: now also SW2.S; no longer J3.+
- net /RESET: no longer J7.S6
- net GND: no longer J7.S8
- net KEY_I2C_SCL: now also U$1PORT5.P5[3]/U4_RXD/I2C0_SCL; no longer U$1PORT0.P0[28]/I2C0_SCL/USB_SCL1
- net KEY_I2C_SDA: now also U$1PORT5.P5[2]/T3_MAT2/I2C0_SDA; no longer U$1PORT0.P0[27]/I2C0_SDA/USB_SDA1
- net SCL: now also R12.2, U$1PORT0.P0[28]/I2C0_SCL/USB_SCL1; no longer R13.2, U$1PORT5.P5[3]/U4_RXD/I2C0_SCL
- net SDA: now also R13.2, U$1PORT0.P0[27]/I2C0_SDA/USB_SDA1; no longer R12.2, U$1PORT5.P5[2]/T3_MAT2/I2C0_SDA
- net TCK/SWDCLK: no longer J7.S3
- net TDI: no longer J7.S5
- net TDO/SWO: no longer J7.S4
- net TMS/SWDIO: no longer J7.S2
Other:
- note added: "Add power switch"
- note removed: "LPC-LINK"
- moved on the sheet: J11, J3, J6, R12, R13

Commit message: Finishing up LCP1788 board
Parts:
- added C33, C34: 0.01uF, rcl:C-EUC0402
- added C35: 0.1uF, rcl:C-EUC0402
- added C36: 10uF, rcl:C-EUC0402
- added C37: 330uF, rcl:C-EUC1206
- added R10, R21, R31: 20K, rcl:R-US_R0402
- added U6: AR1021-RESISTIVE_TOUCH_CONTROLLER, Custom:AR1021-RESISTIVE_TOUCH_CONTROLLER
Connections:
- new net N$35: C33.1, J8.XL, R10.2, U6.X-
- new net N$36: J8.XR, U6.X+
- new net N$37: C34.1, J8.YD, U6.Y-
- new net N$38: J8.YU, U6.Y+
- new net N$39: R21.2, U6.M1
- new net N$40: R10.1, U6.WAKE
- new net N$41: R31.2, U6.M2
- new net TOUCH_INT: U$1PORT2.P2[14]/!EMC_CS2!/I2C1_SDA/T2_CAP0, U6.SDO
- net !BLS0: now also J12.S3; no longer J12.S44
- net !BLS1: now also J12.S20; no longer J12.S46
- net !CAS: now also J12.S21; no longer J12.S48
- net !CS1: now also J12.S33; no longer J12.S42
- net !DYCS0: now also J12.S31; no longer J12.S39
- net !OE: now also J12.S29; no longer J12.S35
- net !RAS: now also J12.S19; no longer J12.S49
- net !WE: now also J12.S2; no longer J12.S37
- net +3V3: now also C35.1, C36.1, J9.S3, J9.S4, U6.VDD
- net +VBAT: now also C37.1
- net A0: now also J12.S27; no longer J12.S2
- net A1: now also J12.S25; no longer J12.S4
- net A10: now also J12.S14; no longer J12.S22
- net A11: now also J12.S12; no longer J12.S24
- net A12: now also J12.S10; no longer J12.S26
- net A13: now also J12.S22; no longer J12.S28
- net A14: now also J12.S8; no longer J12.S30
- net A15: now also J12.S6; no longer J12.S32
- net A16: now also J12.S48; no longer J12.S34
- net A17: now also J12.S13; no longer J12.S36
- net A18: now also J12.S11; no longer J12.S38
- net A19: now also J12.S7; no longer J12.S40
- net A2: now also J12.S23; no longer J12.S6
- net A3: now also J12.S17; no longer J12.S8
- net A4: now also J12.S15; no longer J12.S10
- net A5: now also J12.S9; no longer J12.S12
- net A6: now also J12.S5; no longer J12.S14
- net A7: now also J12.S4; no longer J12.S16
- net A9: now also J12.S16; no longer J12.S20
- net B0: now also J9.S11; no longer J9.S9
- net B1: now also J9.S13; no longer J9.S11
- net B2: now also J9.S8; no longer J9.S13
- net B3: now also J9.S6; no longer J9.S15
- net B4: now also J9.S37; no longer J9.S17
- net B5: now also J9.S39; no longer J9.S19
- net B6: now also J9.S41; no longer J9.S21
- net B7: now also J9.S43; no longer J9.S23
- net CKE: now also J12.S44; no longer J12.S43
- net CLK: now also J12.S46; no longer J12.S41
- net D0: now also J12.S37; no longer J12.S3
- net D1: now also J12.S39; no longer J12.S5
- net D10: now also J12.S45; no longer J12.S23
- net D11: now also J12.S49; no longer J12.S25
- net D12: now also J12.S28; no longer J12.S27
- net D13: now also J12.S32; no longer J12.S29
- net D14: now also J12.S36; no longer J12.S31
- net D15: now also J12.S40; no longer J12.S33
- net D2: now also J12.S43; no longer J12.S7
- net D3: now also J12.S47; no longer J12.S9
- net D4: now also J12.S26; no longer J12.S11
- net D5: now also J12.S30; no longer J12.S13
- net D6: now also J12.S34; no longer J12.S15
- net D7: now also J12.S38; no longer J12.S17
- net D8: now also J12.S35; no longer J12.S19
- net D9: now also J12.S41; no longer J12.S21
- net DQM0: now also J12.S42; no longer J12.S45
- net DQM1: now also J12.S24; no longer J12.S47
- net G0: now also J9.S15; no longer J9.S10
- net G1: now also J9.S5; no longer J9.S12
- net G2: now also J9.S22; no longer J9.S14
- net G3: now also J9.S24; no longer J9.S16
- net G4: now also J9.S16; no longer J9.S18
- net G5: now also J9.S14; no longer J9.S20
- net G6: now also J9.S12; no longer J9.S22
- net G7: now also J9.S10; no longer J9.S24
- net GND: now also C33.2, C34.2, C35.2, C36.2, C37.2, J5.GND, J9.S47, J9.S48, R21.1, R31.1, U6.GND; no longer J5.GND@1
- net LCD_DCLK: now also J9.S21; no longer J9.S5
- net LCD_ENAB_M: now also J9.S25; no longer J9.S7
- net LCD_FP: now also J9.S23; no longer J9.S8
- net LCD_LE: now also J9.S19; no longer J9.S4
- net LCD_LP: now also J9.S27; no longer J9.S6
- net LCD_PWR: now also J9.S17; no longer J9.S3
- net LED1_PWR: now also J9.S30, J9.S32; no longer J9.S26
- net LED2_PWR: now also J9.S36, J9.S38; no longer J9.S28
- net R0: now also J9.S9; no longer J9.S25
- net R1: now also J9.S7; no longer J9.S27
- net R2: now also J9.S33; no longer J9.S29
- net R3: now also J9.S35; no longer J9.S31
- net R4: now also J9.S29; no longer J9.S33
- net R5: now also J9.S31; no longer J9.S35
- net R6: now also J9.S18; no longer J9.S37
- net R7: now also J9.S20; no longer J9.S39
- net SCL: now also U6.SCK/SCL/TX
- net SDA: now also U6.SDI/SDA/RX
- net SD_DET: now also U$1PORT2.P2[15/!EMC_CS3!/I2C1_SCL/T2_CAP1
Other:
- note removed: "Add power switch"
- moved on the sheet: C7, J9
